File: modules/phaser/schematic/phaser_rev_A/phaser_rev_A.kicad_pcb (KiCad board)
At the start: 2 copper layers, 15 parts, among them Q1 2N2978, Q2 2N2978, Q3 2N2978, Q4 2N2978, Q5 2N2978

Commit message: first routing of the PCB added a case study for the phaser
Parts:
- added C11: 22nF, Capacitor_THT:C_Rect_L7.0mm_W2.0mm_P5.00mm, F.Cu at (81.0, 81.5)
- added C12: 22nF, Capacitor_THT:C_Rect_L7.0mm_W2.0mm_P5.00mm, F.Cu at (81.0, 85.0)
- added C13: 10nF, Capacitor_THT:C_Rect_L7.0mm_W2.0mm_P5.00mm, F.Cu at (37.0, 115.8)
- added C14: 22nF, Capacitor_THT:C_Rect_L7.0mm_W2.0mm_P5.00mm, F.Cu at (37.0, 119.3)
- added C15: 22nF, Capacitor_THT:C_Rect_L7.0mm_W2.0mm_P5.00mm, F.Cu at (37.0, 122.9)
- added C16: 22nF, Capacitor_THT:C_Rect_L7.0mm_W2.0mm_P5.00mm, F.Cu at (37.0, 126.5)
- added C17: 22nF, Capacitor_THT:C_Rect_L7.0mm_W2.0mm_P5.00mm, F.Cu at (37.0, 130.0)
- added Q10: BC548, Package_TO_SOT_THT:TO-92L_Inline_Wide, F.Cu at (72.8, 60.4)
- added Q11: BC548, Package_TO_SOT_THT:TO-92L_Inline_Wide, F.Cu at (72.8, 66.0)
- added Q12: BC548, Package_TO_SOT_THT:TO-92L_Inline_Wide, F.Cu at (72.8, 71.7)
- added Q13: BC548, Package_TO_SOT_THT:TO-92L_Inline_Wide, F.Cu at (72.8, 77.3)
- added Q14: BC548, Package_TO_SOT_THT:TO-92L_Inline_Wide, F.Cu at (28.6, 117.3)
- added Q15: BC548, Package_TO_SOT_THT:TO-92L_Inline_Wide, F.Cu at (28.6, 123.0)
- added Q16: BC548, Package_TO_SOT_THT:TO-92L_Inline_Wide, F.Cu at (28.6, 128.6)
- added Q17: BC548, Package_TO_SOT_THT:TO-92L_Inline_Wide, F.Cu at (28.6, 134.2)
- added Q6: BC548, Package_TO_SOT_THT:TO-92L_Inline_Wide, F.Cu at (69.5, 52.0)
- added Q7: BC548, Package_TO_SOT_THT:TO-92L_Inline_Wide, F.Cu at (64.6, 66.0)
- added Q8: BC548, Package_TO_SOT_THT:TO-92L_Inline_Wide, F.Cu at (64.6, 71.7)
- added Q9: BC548, Package_TO_SOT_THT:TO-92L_Inline_Wide, F.Cu at (64.6, 77.3)
- added R1: 100, Resistor_THT:R_Axial_DIN0207_L6.3mm_D2.5mm_P10.16mm_Horizontal, F.Cu at (56.5, 81.7)
- added R2: 100, Resistor_THT:R_Axial_DIN0207_L6.3mm_D2.5mm_P10.16mm_Horizontal, F.Cu at (56.5, 85.8)
- added R3: 100, Resistor_THT:R_Axial_DIN0207_L6.3mm_D2.5mm_P10.16mm_Horizontal, F.Cu at (56.5, 89.8)
- added U1: OPA4376, Package_DIP:DIP-14_W7.62mm_LongPads, F.Cu at (69.2, 120.4)
- Q2, Q3, Q4, Q5: value 2N2978 -> BC548; footprint ProjectLib_Transient:TO-5-6 -> Package_TO_SOT_THT:TO-92L_Inline_Wide
- moved Q5 67.2 mm to (76.5, 45.7), turned to 90 degrees
- moved Q4 64.7 mm to (69.5, 40.6), turned to -90 degrees
- moved C2 56.6 mm to (64.8, 30.5), turned to -90 degrees
- moved Q3 56.3 mm to (76.5, 35.6), turned to 90 degrees
- moved Q2 54.6 mm to (69.5, 30.5), turned to -90 degrees
- moved C3 52.9 mm to (64.8, 40.7), turned to -90 degrees
- moved C4 38.8 mm to (81.3, 45.7), turned to 90 degrees
- moved C1 38.4 mm to (81.3, 35.5), turned to 90 degrees
- moved Q1 35.5 mm to (71.2, 85.2)
Connections:
- C1 pad 1: Net-(Q1A-B1) -> Net-(Q2-B)
- C1 pad 2: Net-(Q1B-E2) -> Net-(Q3-E)
- C10 pad 1: Net-(Q4B-E2) -> Net-(Q10-B)
- C10 pad 2: Net-(Q5B-E2) -> Net-(Q11-E)
- C2 pad 1: Net-(Q1A-C1) -> Net-(Q2-C)
- C2 pad 2: Net-(Q1A-E1) -> Net-(Q2-E)
- C3 pad 1: Net-(Q1A-E1) -> Net-(Q2-E)
- C3 pad 2: Net-(Q2A-E1) -> Net-(Q4-E)
- C4 pad 1: Net-(Q1B-E2) -> Net-(Q3-E)
- C4 pad 2: Net-(Q2B-E2) -> Net-(Q5-E)
- C5 pad 1: Net-(Q2A-E1) -> Net-(Q4-E)
- C5 pad 2: Net-(Q3A-E1) -> Net-(Q6-E)
- C6 pad 1: Net-(Q2B-E2) -> Net-(Q5-E)
- C6 pad 2: Net-(Q3B-E2) -> Net-(Q7-E)
- C7 pad 1: Net-(Q3A-E1) -> Net-(Q6-E)
- C7 pad 2: Net-(Q4A-E1) -> Net-(Q10-C)
- C8 pad 1: Net-(Q3B-E2) -> Net-(Q7-E)
- C8 pad 2: Net-(Q4B-E2) -> Net-(Q10-B)
- C9 pad 1: Net-(Q4A-E1) -> Net-(Q10-C)
- C9 pad 2: Net-(Q5A-E1) -> Net-(Q10-E)
- Q1 pad 3: Net-(Q1A-C1) -> Net-(Q17-E)
- Q1 pad 5: Net-(Q1B-E2) -> Net-(Q1A-E1)
- Q1 pad 6: Net-(Q1A-C1) -> Net-(Q1A-B1)
- Q1 pad 7: Net-(Q1A-B1) -> Net-(Q16-E)
- Q2 pad 1: Net-(Q2A-E1) -> Net-(Q2-C)
- Q2 pad 2: Net-(Q1B-E2) -> Net-(Q2-B)
- Q2 pad 3: Net-(Q1A-E1) -> Net-(Q2-E)
- Q3 pad 1: Net-(Q3A-E1) -> Net-(Q2-B)
- Q3 pad 2: Net-(Q2B-E2) -> Net-(Q2-C)
- Q3 pad 3: Net-(Q2A-E1) -> Net-(Q3-E)
- Q4 pad 1: Net-(Q4A-E1) -> Net-(Q2-E)
- Q4 pad 2: Net-(Q3B-E2) -> Net-(Q3-E)
- Q4 pad 3: Net-(Q3A-E1) -> Net-(Q4-E)
- Q5 pad 1: Net-(Q5A-E1) -> Net-(Q3-E)
- Q5 pad 2: Net-(Q4B-E2) -> Net-(Q2-E)
- Q5 pad 3: Net-(Q4A-E1) -> Net-(Q5-E)
Routing:
- net Net-(Q3-E): track 0.00 -> 39.0 mm
- net Net-(Q2-E): track 0.00 -> 22.6 mm
- net Net-(Q2-B): track 0.00 -> 12.8 mm
- net Net-(Q2-C): track 0.00 -> 12.8 mm
- net Net-(Q5-E): track 0.00 -> 4.85 mm
- net Net-(Q4-E): track 0.00 -> 4.79 mm
